File: SP3485.kicad_sch (KiCad schematic)
At the start: 17 parts, among them J3 Conn_01x02_Male, U2 SP3485EN

Commit message: finish some unconnect pins, draw edge cut board
Parts:
- D1, D2, D3: value D_TVS -> SMAJ28A
- F2, F3: value Polyfuse -> MF-MSMF050-2
Connections:
- net RS485.DERE renamed RS485_input.DERE
- net RS485.RX renamed RS485_input.RX
- net RS485.TX renamed RS485_input.TX
Changed lines of the file:
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@@
 	(wire
 		(pts
-			(xy 76.2 96.52) (xy 87.63 96.52)
+			(xy 76.2 96.52) (xy 91.44 96.52)
 		)
 		(stroke
@@
 	(wire
 		(pts
-			(xy 76.2 101.6) (xy 87.63 101.6)
+			(xy 76.2 101.6) (xy 91.44 101.6)
 		)
 		(stroke
@@
 	(wire
 		(pts
-			(xy 76.2 99.06) (xy 90.17 99.06)
+			(xy 76.2 99.06) (xy 93.98 99.06)
 		)
 		(stroke
@@
 		)
 	)
-	(label "RS485.RX"
-		(at 87.63 101.6 180)
+	(label "RS485_input.RX"
+		(at 76.2 74.93 180)
+		(fields_autoplaced yes)
+		(effects
+			(font
+				(size 1.27 1.27)
+			)
+			(justify right bottom)
+		)
+	)
+	(label "RS485_input.RX"
+		(at 91.44 101.6 180)
 		(fields_autoplaced yes)
 		(effects
@@
 		)
 	)
-	(label "RS485.TX"
+	(label "RS485_input.DERE"
+		(at 93.98 99.06 180)
+		(fields_autoplaced yes)
+		(effects
+			(font
+				(size 1.27 1.27)
+			)
+			(justify right bottom)
+		)
+	)
+	(label "RS485_input.DERE"
+		(at 76.2 80.01 180)
+		(fields_autoplaced yes)
+		(effects
+			(font
+				(size 1.27 1.27)
+			)
+			(justify right bottom)
+		)
+	)
+	(label "RS485_input.TX"
 		(at 76.2 85.09 180)
 		(fields_autoplaced yes)
@@
 		)
 	)
-	(label "RS485.RX"
-		(at 76.2 74.93 180)
-		(fields_autoplaced yes)
-		(effects
-			(font
-				(size 1.27 1.27)
-			)
-			(justify right bottom)
-		)
-	)
-	(label "RS485.DERE"
-		(at 90.17 99.06 180)
-		(fields_autoplaced yes)
-		(effects
-			(font
-				(size 1.27 1.27)
-			)
-			(justify right bottom)
-		)
-	)
-	(label "RS485.DERE"
-		(at 76.2 80.01 180)
-		(fields_autoplaced yes)
-		(effects
-			(font
-				(size 1.27 1.27)
-			)
-			(justify right bottom)
-		)
-	)
-	(label "RS485.TX"
-		(at 87.63 96.52 180)
+	(label "RS485_input.TX"
+		(at 91.44 96.52 180)
 		(fields_autoplaced yes)
 		(effects
@@
 			)
 		)
-		(property "Value" "D_TVS"
+		(property "Value" "SMAJ28A"
 			(at 170.18 92.7099 90)
 			(effects
@@
 			)
 		)
-		(property "Value" "D_TVS"
+		(property "Value" "SMAJ28A"
 			(at 170.18 81.2799 90)
 			(effects
@@
 			)
 		)
-		(property "Value" "Polyfuse"
+		(property "Value" "MF-MSMF050-2"
 			(at 185.42 87.63 90)
 			(effects
@@
 			)
 		)
-		(property "Value" "Polyfuse"
+		(property "Value" "MF-MSMF050-2"
 			(at 185.42 71.12 90)
 			(effects
@@
 			)
 		)
-		(property "Value" "D_TVS"
+		(property "Value" "SMAJ28A"
 			(at 150.495 93.345 90)
 			(effects

Commit message: Add LORA, SDcard and Volt to 4_20mA scheamtic
Parts:
- renumbered D1 to D5, D2 to D6, D3 to D7, J3 to J6
Connections:
- net 3.3V_Supply renamed 3V3
- net Digital_GND renamed GND
Changed lines of the file:
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@@
 		)
 	)
-	(hierarchical_label "Digital_GND"
+	(hierarchical_label "GND"
 		(shape passive)
 		(at 95.25 63.5 180)
@@
 		)
 	)
-	(hierarchical_label "3.3V_Supply"
+	(hierarchical_label "3V3"
 		(shape passive)
 		(at 130.81 57.15 90)
@@
 		)
 	)
-	(hierarchical_label "3.3V_Supply"
+	(hierarchical_label "3V3"
 		(shape passive)
 		(at 109.22 60.96 90)
@@
 		)
 	)
-	(hierarchical_label "Digital_GND"
+	(hierarchical_label "GND"
 		(shape passive)
 		(at 109.22 104.14 270)
@@
 		(dnp no)
 		(fields_autoplaced yes)
-		(property "Reference" "D3"
+		(property "Reference" "D7"
 			(at 170.18 90.1699 90)
 			(effects
@@
 			(project "DongTamV2"
 				(path "/2303d546-b88a-4ab0-aee1-26e3b32ac9d7/8af8cae9-6834-4c4e-95b1-3f358a1db5d8"
-					(reference "D3")
+					(reference "D7")
 					(unit 1)
 				)
@@
 		(dnp no)
 		(fields_autoplaced yes)
-		(property "Reference" "D2"
+		(property "Reference" "D6"
 			(at 170.18 78.7399 90)
 			(effects
@@
 			(project "DongTamV2"
 				(path "/2303d546-b88a-4ab0-aee1-26e3b32ac9d7/8af8cae9-6834-4c4e-95b1-3f358a1db5d8"
-					(reference "D2")
+					(reference "D6")
 					(unit 1)
 				)
@@
 		(on_board yes)
 		(dnp no)
-		(property "Reference" "J3"
+		(property "Reference" "J6"
 			(at 156.21 56.5149 90)
 			(effects
@@
 			(project "DongTamV2"
 				(path "/2303d546-b88a-4ab0-aee1-26e3b32ac9d7/8af8cae9-6834-4c4e-95b1-3f358a1db5d8"
-					(reference "J3")
+					(reference "J6")
 					(unit 1)
 				)
@@
 		(on_board yes)
 		(dnp no)
-		(property "Reference" "D1"
+		(property "Reference" "D5"
 			(at 150.495 90.805 90)
 			(effects
@@
 			(project "DongTamV2"
 				(path "/2303d546-b88a-4ab0-aee1-26e3b32ac9d7/8af8cae9-6834-4c4e-95b1-3f358a1db5d8"
-					(reference "D1")
-					(unit 1)
-				)
+					(reference "D5")
+					(unit 1)
+				)
