File: IDC14pin.kicad_sch (KiCad schematic)
At the start: 16 parts, among them J9 IDC_02x07, Q1 N_Mosfet, Q2 N_Mosfet, Q3 N_Mosfet, Q4 N_Mosfet, Q5 N_Mosfet

Commit message: finish some unconnect pins, draw edge cut board
Parts:
- Q1, Q2, Q3, Q4, Q5: value N_Mosfet -> SI2302/BSS138
Changed lines of the file:
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@@
 			)
 		)
-		(property "Value" "N_Mosfet"
+		(property "Value" "SI2302/BSS138"
 			(at 55.88 121.285 0)
 			(effects
@@
 			)
 		)
-		(property "Value" "N_Mosfet"
+		(property "Value" "SI2302/BSS138"
 			(at 69.85 91.44 0)
 			(effects
@@
 			)
 		)
-		(property "Value" "N_Mosfet"
+		(property "Value" "SI2302/BSS138"
 			(at 77.47 96.52 0)
 			(effects
@@
 			)
 		)
-		(property "Value" "N_Mosfet"
+		(property "Value" "SI2302/BSS138"
 			(at 63.5 126.365 0)
 			(effects
@@
 			)
 		)
-		(property "Value" "N_Mosfet"
+		(property "Value" "SI2302/BSS138"
 			(at 71.755 132.715 0)
 			(effects

Commit message: Add LORA, SDcard and Volt to 4_20mA scheamtic
Parts:
- renumbered J9 to J11, R38 to R41, R39 to R42, R40 to R43, R41 to R44, R42 to R45, R43 to R46, R44 to R47, R45 to R48, R46 to R49, R47 to R50
Changed lines of the file:
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@@
 		(dnp no)
 		(fields_autoplaced yes)
-		(property "Reference" "#PWR042"
+		(property "Reference" "#PWR047"
 			(at 113.03 45.72 0)
 			(effects
@@
 			(project "DongTamV2"
 				(path "/2303d546-b88a-4ab0-aee1-26e3b32ac9d7/1fc168b8-b0db-4323-90d7-bec14ecfc338"
-					(reference "#PWR042")
+					(reference "#PWR047")
 					(unit 1)
 				)
@@
 		(on_board yes)
 		(dnp no)
-		(property "Reference" "R43"
+		(property "Reference" "R46"
 			(at 93.345 110.49 0)
 			(effects
@@
 			(project "DongTamV2"
 				(path "/2303d546-b88a-4ab0-aee1-26e3b32ac9d7/1fc168b8-b0db-4323-90d7-bec14ecfc338"
-					(reference "R43")
+					(reference "R46")
 					(unit 1)
 				)
@@
 		(dnp no)
 		(fields_autoplaced yes)
-		(property "Reference" "#PWR038"
+		(property "Reference" "#PWR043"
 			(at 69.215 45.72 0)
 			(effects
@@
 			(project "DongTamV2"
 				(path "/2303d546-b88a-4ab0-aee1-26e3b32ac9d7/1fc168b8-b0db-4323-90d7-bec14ecfc338"
-					(reference "#PWR038")
+					(reference "#PWR043")
 					(unit 1)
 				)
@@
 		(on_board yes)
 		(dnp no)
-		(property "Reference" "R38"
+		(property "Reference" "R41"
 			(at 52.705 111.125 0)
 			(effects
@@
 			(project "DongTamV2"
 				(path "/2303d546-b88a-4ab0-aee1-26e3b32ac9d7/1fc168b8-b0db-4323-90d7-bec14ecfc338"
-					(reference "R38")
+					(reference "R41")
 					(unit 1)
 				)
@@
 		(on_board yes)
 		(dnp no)
-		(property "Reference" "R41"
+		(property "Reference" "R44"
 			(at 61.595 83.82 0)
 			(effects
@@
 			(project "DongTamV2"
 				(path "/2303d546-b88a-4ab0-aee1-26e3b32ac9d7/1fc168b8-b0db-4323-90d7-bec14ecfc338"
-					(reference "R41")
+					(reference "R44")
 					(unit 1)
 				)
@@
 		(on_board yes)
 		(dnp no)
-		(property "Reference" "R47"
+		(property "Reference" "R50"
 			(at 109.855 111.125 0)
 			(effects
@@
 			(project "DongTamV2"
 				(path "/2303d546-b88a-4ab0-aee1-26e3b32ac9d7/1fc168b8-b0db-4323-90d7-bec14ecfc338"
-					(reference "R47")
+					(reference "R50")
 					(unit 1)
 				)
@@
 		(dnp no)
 		(fields_autoplaced yes)
-		(property "Reference" "J9"
+		(property "Reference" "J11"
 			(at 83.82 24.13 0)
 			(effects
@@
 			(project "DongTamV2"
 				(path "/2303d546-b88a-4ab0-aee1-26e3b32ac9d7/1fc168b8-b0db-4323-90d7-bec14ecfc338"
-					(reference "J9")
+					(reference "J11")
 					(unit 1)
 				)
@@
 		(on_board yes)
 		(dnp no)
-		(property "Reference" "#PWR040"
+		(property "Reference" "#PWR045"
 			(at 100.33 81.915 0)
 			(effects
@@
 			(project "DongTamV2"
 				(path "/2303d546-b88a-4ab0-aee1-26e3b32ac9d7/1fc168b8-b0db-4323-90d7-bec14ecfc338"
-					(reference "#PWR040")
+					(reference "#PWR045")
 					(unit 1)
 				)
@@
 		(on_board yes)
 		(dnp no)
-		(property "Reference" "R39"
+		(property "Reference" "R42"
 			(at 57.785 111.125 0)
 			(effects
@@
 			(project "DongTamV2"
 				(path "/2303d546-b88a-4ab0-aee1-26e3b32ac9d7/1fc168b8-b0db-4323-90d7-bec14ecfc338"
-					(reference "R39")
+					(reference "R42")
 					(unit 1)
 				)
@@
 		(on_board yes)
 		(dnp no)
-		(property "Reference" "R44"
+		(property "Reference" "R47"
 			(at 93.98 83.82 0)
 			(effects
@@
 			(project "DongTamV2"
 				(path "/2303d546-b88a-4ab0-aee1-26e3b32ac9d7/1fc168b8-b0db-4323-90d7-bec14ecfc338"
-					(reference "R44")
+					(reference "R47")
 					(unit 1)
 				)
@@
 		(on_board yes)
 		(dnp no)
-		(property "Reference" "#PWR036"
+		(property "Reference" "#PWR041"
 			(at 52.07 30.48 0)
 			(effects
@@
 			(project "DongTamV2"
 				(path "/2303d546-b88a-4ab0-aee1-26e3b32ac9d7/1fc168b8-b0db-4323-90d7-bec14ecfc338"
-					(reference "#PWR036")
+					(reference "#PWR041")
 					(unit 1)
 				)
@@
 		(dnp no)
 		(fields_autoplaced yes)
-		(property "Reference" "#PWR043"
+		(property "Reference" "#PWR048"
 			(at 103.505 30.48 0)
 			(effects
@@
 			(project "DongTamV2"
 				(path "/2303d546-b88a-4ab0-aee1-26e3b32ac9d7/1fc168b8-b0db-4323-90d7-bec14ecfc338"
-					(reference "#PWR043")
+					(reference "#PWR048")
 					(unit 1)
 				)
@@
 		(on_board yes)
 		(dnp no)
-		(property "Reference" "R46"
+		(property "Reference" "R49"
 			(at 104.14 111.125 0)
 			(effects
@@
 			(project "DongTamV2"
 				(path "/2303d546-b88a-4ab0-aee1-26e3b32ac9d7/1fc168b8-b0db-4323-90d7-bec14ecfc338"
-					(reference "R46")
+					(reference "R49")
 					(unit 1)
 				)
@@
 		(dnp no)
 		(fields_autoplaced yes)
-		(property "Reference" "R45"
+		(property "Reference" "R48"
 			(at 104.14 83.8199 0)
 			(effects
@@
 			(project "DongTamV2"
 				(path "/2303d546-b88a-4ab0-aee1-26e3b32ac9d7/1fc168b8-b0db-4323-90d7-bec14ecfc338"
-					(reference "R45")
+					(reference "R48")
 					(unit 1)
 				)
@@
 		(dnp no)
 		(fields_autoplaced yes)
-		(property "Reference" "R42"
+		(property "Reference" "R45"
 			(at 71.755 83.8199 0)
 			(effects
@@
 			(project "DongTamV2"
 				(path "/2303d546-b88a-4ab0-aee1-26e3b32ac9d7/1fc168b8-b0db-4323-90d7-bec14ecfc338"
-					(reference "R42")
+					(reference "R45")
 					(unit 1)
 				)
@@
 		(on_board yes)
 		(dnp no)
-		(property "Reference" "#PWR039"
+		(property "Reference" "#PWR044"
 			(at 76.2 81.915 0)
 			(effects
@@
 			(project "DongTamV2"
 				(path "/2303d546-b88a-4ab0-aee1-26e3b32ac9d7/1fc168b8-b0db-4323-90d7-bec14ecfc338"
-					(reference "#PWR039")
+					(reference "#PWR044")
 					(unit 1)
 				)
@@
 		(on_board yes)
 		(dnp no)
-		(property "Reference" "#PWR041"
+		(property "Reference" "#PWR046"
 			(at 103.505 111.76 0)
 			(effects
@@
 			(project "DongTamV2"
 				(path "/2303d546-b88a-4ab0-aee1-26e3b32ac9d7/1fc168b8-b0db-4323-90d7-bec14ecfc338"
-					(reference "#PWR041")
+					(reference "#PWR046")
 					(unit 1)
 				)
@@
 		(on_board yes)
 		(dnp no)
-		(property "Reference" "R40"
+		(property "Reference" "R43"
 			(at 62.23 111.125 0)
 			(effects
@@
 			(project "DongTamV2"
 				(path "/2303d546-b88a-4ab0-aee1-26e3b32ac9d7/1fc168b8-b0db-4323-90d7-bec14ecfc338"
-					(reference "R40")
+					(reference "R43")
 					(unit 1)
 				)
@@
 		(on_board yes)
 		(dnp no)
-		(property "Reference" "#PWR037"
+		(property "Reference" "#PWR042"
 			(at 62.23 111.76 0)
 			(effects
@@
 			(project "DongTamV2"
 				(path "/2303d546-b88a-4ab0-aee1-26e3b32ac9d7/1fc168b8-b0db-4323-90d7-bec14ecfc338"
-					(reference "#PWR037")
-					(unit 1)
-				)
+					(reference "#PWR042")
+					(unit 1)
+				)

Commit message: layout p1
Connections:
- net +3V3 renamed +3.3V
Changed lines of the file:
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@@
+	)
+	(symbol
+		(lib_id "power:+3.3V")
+		(at 76.2 78.105 0)
+		(unit 1)
+		(exclude_from_sim no)
+		(in_bom yes)
+		(on_board yes)
+		(dnp no)
+		(fields_autoplaced yes)
+		(property "Reference" "#PWR042"
+			(at 76.2 81.915 0)
+			(effects
+				(font
+					(size 1.27 1.27)
+				)
+				(hide yes)
+			)
+		)
+		(property "Value" "+3.3V"
+			(at 76.2 73.025 0)
+			(effects
+				(font
+					(size 1.27 1.27)
+				)
+			)
+		)
+		(property "Footprint" ""
+			(at 76.2 78.105 0)
+			(effects
+				(font
+					(size 1.27 1.27)
+				)
+				(hide yes)
+			)
+		)
+		(property "Datasheet" ""
+			(at 76.2 78.105 0)
+			(effects
+				(font
+					(size 1.27 1.27)
+				)
+				(hide yes)
+			)
+		)
+		(property "Description" "Power symbol creates a global label with name \"+3.3V\""
+			(at 76.2 78.105 0)
+			(effects
+				(font
+					(size 1.27 1.27)
+				)
+				(hide yes)
+			)
+		)
+		(pin "1"
+		)
+		(instances
+			(project "DongTamV2"
+				(path "/2303d546-b88a-4ab0-aee1-26e3b32ac9d7/1fc168b8-b0db-4323-90d7-bec14ecfc338"
+					(reference "#PWR042")
+					(unit 1)
+				)
+			)
+		)
 	)
 	(symbol
@@
 	)
 	(symbol
-		(lib_id "power:+3V3")
+		(lib_id "power:+3.3V")
 		(at 107.315 30.48 270)
 		(unit 1)
@@
 		(dnp no)
 		(fields_autoplaced yes)
-		(property "Reference" "#PWR048"
+		(property "Reference" "#PWR044"
 			(at 103.505 30.48 0)
 			(effects
@@
 			)
 		)
-		(property "Value" "+3V3"
-			(at 111.125 30.4799 90)
+		(property "Value" "+3.3V"
+			(at 110.49 30.4799 90)
 			(effects
 				(font
@@
 			)
 		)
-		(property "Description" ""
+		(property "Description" "Power symbol creates a global label with name \"+3.3V\""
 			(at 107.315 30.48 0)
 			(effects
@@
 			(project "DongTamV2"
 				(path "/2303d546-b88a-4ab0-aee1-26e3b32ac9d7/1fc168b8-b0db-4323-90d7-bec14ecfc338"
-					(reference "#PWR048")
-					(unit 1)
-				)
-			)
-			(project "dongtam"
-				(path "/6833aec4-3d1d-4261-9b3e-f0452b565dd3/b0d5c22f-fe0a-4806-9983-e193fa74270b"
-					(reference "#PWR0181")
+					(reference "#PWR044")
+					(unit 1)
+				)
+			)
+		)
+	)
+	(symbol
+		(lib_id "power:+3.3V")
+		(at 62.23 107.95 0)
+		(unit 1)
+		(exclude_from_sim no)
+		(in_bom yes)
+		(on_board yes)
+		(dnp no)
+		(fields_autoplaced yes)
+		(property "Reference" "#PWR035"
+			(at 62.23 111.76 0)
+			(effects
+				(font
+					(size 1.27 1.27)
+				)
+				(hide yes)
+			)
+		)
+		(property "Value" "+3.3V"
+			(at 62.23 102.87 0)
+			(effects
+				(font
+					(size 1.27 1.27)
+				)
+			)
+		)
+		(property "Footprint" ""
+			(at 62.23 107.95 0)
+			(effects
+				(font
+					(size 1.27 1.27)
+				)
+				(hide yes)
+			)
+		)
+		(property "Datasheet" ""
+			(at 62.23 107.95 0)
+			(effects
+				(font
+					(size 1.27 1.27)
+				)
+				(hide yes)
+			)
+		)
+		(property "Description" "Power symbol creates a global label with name \"+3.3V\""
+			(at 62.23 107.95 0)
+			(effects
+				(font
+					(size 1.27 1.27)
+				)
+				(hide yes)
+			)
+		)
+		(pin "1"
+		)
+		(instances
+			(project "DongTamV2"
+				(path "/2303d546-b88a-4ab0-aee1-26e3b32ac9d7/1fc168b8-b0db-4323-90d7-bec14ecfc338"
+					(reference "#PWR035")
 					(unit 1)
 				)
@@
 	)
 	(symbol
-		(lib_id "power:+3V3")
-		(at 76.2 78.105 0)
-		(unit 1)
-		(exclude_from_sim no)
-		(in_bom yes)
-		(on_board yes)
-		(dnp no)
-		(property "Reference" "#PWR044"
-			(at 76.2 81.915 0)
-			(effects
-				(font
-					(size 1.27 1.27)
-				)
-				(hide yes)
-			)
-		)
-		(property "Value" "+3V3"
-			(at 78.105 76.835 0)
-			(effects
-				(font
-					(size 1.27 1.27)
-				)
-				(justify left)
-			)
-		)
-		(property "Footprint" ""
-			(at 76.2 78.105 0)
-			(effects
-				(font
-					(size 1.27 1.27)
-				)
-				(hide yes)
-			)
-		)
-		(property "Datasheet" ""
-			(at 76.2 78.105 0)
-			(effects
-				(font
-					(size 1.27 1.27)
-				)
-				(hide yes)
-			)
-		)
-		(property "Description" ""
-			(at 76.2 78.105 0)
-			(effects
-				(font
-					(size 1.27 1.27)
-				)
-				(hide yes)
-			)
-		)
-		(pin "1"
-		)
-		(instances
-			(project "DongTamV2"
-				(path "/2303d546-b88a-4ab0-aee1-26e3b32ac9d7/1fc168b8-b0db-4323-90d7-bec14ecfc338"
-					(reference "#PWR044")
-					(unit 1)
-				)
-			)
-			(project "dongtam"
-				(path "/6833aec4-3d1d-4261-9b3e-f0452b565dd3/b0d5c22f-fe0a-4806-9983-e193fa74270b"
-					(reference "#PWR0178")
-					(unit 1)
-				)
-			)
-		)
-	)
-	(symbol
 		(lib_id "IVS_SYMBOLS:N_Mosfet")
 		(at 85.725 131.445 270)
@@
 					(unit 1)
 				)
-			)
-		)
-	)
-	(symbol
-		(lib_id "power:+3V3")
-		(at 62.23 107.95 0)
-		(unit 1)
-		(exclude_from_sim no)
-		(in_bom yes)
-		(on_board yes)
-		(dnp no)
-		(property "Reference" "#PWR042"
-			(at 62.23 111.76 0)
-			(effects
-				(font
-					(size 1.27 1.27)
-				)
-				(hide yes)
-			)
-		)
-		(property "Value" "+3V3"
-			(at 64.135 106.68 0)
-			(effects
-				(font
-					(size 1.27 1.27)
-				)
-				(justify left)
-			)
-		)
-		(property "Footprint" ""
-			(at 62.23 107.95 0)
-			(effects
-				(font
-					(size 1.27 1.27)
-				)
-				(hide yes)
-			)
-		)
-		(property "Datasheet" ""
-			(at 62.23 107.95 0)
-			(effects
-				(font
-					(size 1.27 1.27)
-				)
-				(hide yes)
-			)
-		)
-		(property "Description" ""
-			(at 62.23 107.95 0)
-			(effects
-				(font
-					(size 1.27 1.27)
-				)
-				(hide yes)
-			)
-		)
-		(pin "1"
-		)
-		(instances
-			(project "DongTamV2"
-				(path "/2303d546-b88a-4ab0-aee1-26e3b32ac9d7/1fc168b8-b0db-4323-90d7-bec14ecfc338"
-					(reference "#PWR042")
-					(unit 1)
-				)
-			)
-			(project "dongtam"
-				(path "/6833aec4-3d1d-4261-9b3e-f0452b565dd3/b0d5c22f-fe0a-4806-9983-e193fa74270b"
-					(reference "#PWR0103")
-					(unit 1)
-				)
