File: ReadValveState.kicad_sch (KiCad schematic)
At the start: 4 parts, among them U16 74HC165, U17 74HC165

Commit message: finish some unconnect pins, draw edge cut board
Connections:
- net 74HC165.DATA renamed InputExpanderPort.DATA
- net 74HC165.LOAD renamed InputExpanderPort.LOAD
- net 74HC165.SCK renamed InputExpanderPort.SCK
Changed lines of the file:
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@@
 	(wire
 		(pts
-			(xy 184.785 48.895) (xy 175.26 48.895)
+			(xy 184.785 48.895) (xy 183.515 48.895)
 		)
 		(stroke
@@
 		)
 	)
-	(label "74HC165.SCK"
-		(at 111.125 95.885 180)
-		(fields_autoplaced yes)
-		(effects
-			(font
-				(size 1.27 1.27)
-			)
-			(justify right bottom)
-		)
-	)
-	(label "74HC165.DATA"
-		(at 175.26 48.895 180)
-		(fields_autoplaced yes)
-		(effects
-			(font
-				(size 1.27 1.27)
-			)
-			(justify right bottom)
-		)
-	)
 	(label "VO_8"
 		(at 219.075 69.215 180)
@@
 		)
 	)
+	(label "InputExpanderPort.LOAD"
+		(at 111.125 98.425 180)
+		(fields_autoplaced yes)
+		(effects
+			(font
+				(size 1.27 1.27)
+			)
+			(justify right bottom)
+		)
+	)
 	(label "VO_3"
 		(at 219.075 56.515 180)
@@
 		)
 	)
+	(label "InputExpanderPort.SCK"
+		(at 111.125 95.885 180)
+		(fields_autoplaced yes)
+		(effects
+			(font
+				(size 1.27 1.27)
+			)
+			(justify right bottom)
+		)
+	)
 	(label "VO_16"
 		(at 154.305 69.215 180)
@@
 		)
 	)
-	(label "74HC165.SCK"
+	(label "InputExpanderPort.SCK"
 		(at 121.285 151.765 180)
 		(fields_autoplaced yes)
@@
 		)
 	)
+	(label "InputExpanderPort.DATA"
+		(at 183.515 48.895 180)
+		(fields_autoplaced yes)
+		(effects
+			(font
+				(size 1.27 1.27)
+			)
+			(justify right bottom)
+		)
+	)
 	(label "VO_13"
 		(at 154.305 61.595 180)
@@
 		)
 	)
-	(label "74HC165.LOAD"
+	(label "InputExpanderPort.LOAD"
 		(at 121.285 154.305 180)
-		(fields_autoplaced yes)
-		(effects
-			(font
-				(size 1.27 1.27)
-			)
-			(justify right bottom)
-		)
-	)
-	(label "74HC165.LOAD"
-		(at 111.125 98.425 180)
 		(fields_autoplaced yes)
 		(effects
@@
 		)
 	)
-	(label "74HC165.DATA"
+	(label "InputExpanderPort.DATA"
 		(at 121.285 149.225 180)
 		(fields_autoplaced yes)

Commit message: Add LORA, SDcard and Volt to 4_20mA scheamtic
Parts:
- renumbered C38 to C36, U17 to U15
Connections:
- net VCC renamed 5V
Changed lines of the file:
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@@
 		)
 	)
-	(hierarchical_label "VCC"
+	(hierarchical_label "5V"
 		(shape passive)
 		(at 135.255 36.83 90)
@@
 		)
 	)
-	(hierarchical_label "VCC"
+	(hierarchical_label "5V"
 		(shape passive)
 		(at 197.485 36.83 90)
@@
 		(dnp no)
 		(fields_autoplaced yes)
-		(property "Reference" "U17"
+		(property "Reference" "U15"
 			(at 133.2356 41.275 0)
 			(effects
@@
 			(project "DongTamV2"
 				(path "/2303d546-b88a-4ab0-aee1-26e3b32ac9d7/b95e5759-15dd-414c-a82d-930819dc6d8f"
-					(reference "U17")
+					(reference "U15")
 					(unit 1)
 				)
@@
 		(dnp no)
 		(fields_autoplaced yes)
-		(property "Reference" "C38"
+		(property "Reference" "C36"
 			(at 141.605 32.385 90)
 			(effects
@@
 			(project "DongTamV2"
 				(path "/2303d546-b88a-4ab0-aee1-26e3b32ac9d7/b95e5759-15dd-414c-a82d-930819dc6d8f"
-					(reference "C38")
+					(reference "C36")
 					(unit 1)
 				)

Commit message: Layout p2, fix Analog VCC and GND for opamp circuit
Connections:
- net 74HC165_CascadeDATA: now reaches U15.9 (Q7), U16.10 (DS)
Changed lines of the file:
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@@
+		)
+	)
+	(label "74HC165_CascadeDATA"
+		(at 196.215 27.94 0)
+		(fields_autoplaced yes)
+		(effects
+			(font
+				(size 1.27 1.27)
+			)
+			(justify left bottom)
 		)
 	)
