File: DongTamV2.kicad_pcb (KiCad board)
At the start: 2 copper layers, 254 x 135 mm, 288 parts, among them J1 KF128, J10 Conn_01x05_Male, J11 IDC_02x07, J12 USB_C_Receptacle, J13 KF-5.08-8-V, J14 KF-5.08-8-V, J15 KF-5.08-8-V, J16 KF-5.08-8-V, J17 Micro_SD_Card_Det1, J18 HT3.96mm-3P, J2 KF128, J3 KF128, J4 KF128, J5 KF128, J6 Conn_01x02_Male, J7 Conn_02x03_Odd_Even, J9 Conn_01x05_Male, Q1 SI2302/BSS138, Q10 SI2302, Q11 SI2302, Q12 SI2302, Q13 SI2302, Q14 SI2302, Q15 SI2302, Q16 SI2302, Q17 SI2302, Q18 SI2302, Q19 SI2302, Q2 SI2302/BSS138, Q20 SI2302, Q21 SI2302, Q22 MMBT3904, Q3 SI2302/BSS138, Q4 SI2302/BSS138, Q5 SI2302/BSS138, Q6 SI2302, Q7 SI2302, Q8 SI2302, Q9 SI2302, SW1 PTS810, SW2 PTS810, SW3 PTS810, U1 AM22-24W2405V, U10 LD1117, U11 LM324, U12 LM324, U13 LM324, U14 LM324, U15 74HC165, U16 74HC165, U17 RF_Module_Ai-Thinker-Ra-02, U18 LM324, U19 LM317_TO-252, U2 SP3485EN, U20 TL431, U21 MCP41010, U3 MCU_STM32F103C8Tx, U4 ESP32-WROOM-32, U5 PCF8563TS, U6 AMS5915, U7 74HC595, U8 74HC595, U9 USBLC6-2SC6, Y1 16MHz, Y2 MC-306

Commit message: Complete to pull
Routing:
- net Net-(J2-Pin_1): track 0.00 -> 6.31 mm
- net Net-(J3-Pin_1): track 0.00 -> 6.06 mm
- net +24V: track 67.8 -> 69.2 mm
Changed lines of the file:
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@@
 		(tags "Diode")
 		(property "Reference" "D18"
-			(at 2.7 0 360)
+			(at 2.7 0 0)
 			(layer "F.SilkS")
 			(hide yes)
@@
 		)
 		(property "Value" "1N4007"
-			(at 0.1 1.475 360)
+			(at 0.1 1.475 0)
 			(layer "F.Fab")
 			(effects
@@
 		(tags "Diode")
 		(property "Reference" "D16"
-			(at 2.7 0 360)
+			(at 2.7 0 0)
 			(layer "F.SilkS")
 			(hide yes)
@@
 		)
 		(property "Value" "1N4007"
-			(at 0.1 1.475 360)
+			(at 0.1 1.475 0)
 			(layer "F.Fab")
 			(effects
@@
 		)
 		(property "Value" "LM324"
-			(at -0.29 5.74 360)
+			(at -0.29 5.74 0)
 			(layer "F.Fab")
 			(effects
@@
 		)
 		(property "Value" "LM324"
-			(at -0.29 5.74 360)
+			(at -0.29 5.74 0)
 			(layer "F.Fab")
 			(effects
@@
 		(at 192.115156 137.6925)
 		(property "Reference" "J16"
-			(at 17.78 -5.46 360)
+			(at 17.78 -5.46 0)
 			(layer "F.SilkS")
 			(effects
@@
 		)
 		(property "Value" "KF-5.08-8-V"
-			(at 17.78 5.11 360)
+			(at 17.78 5.11 0)
 			(layer "F.Fab")
 			(effects
@@
 		)
 		(fp_text user "${REFERENCE}"
-			(at 17.78 -5.46 360)
+			(at 17.78 -5.46 0)
 			(layer "F.Fab")
 			(effects
@@
 		(tags "Diode")
 		(property "Reference" "D22"
-			(at 2.7 0 360)
+			(at 2.7 0 0)
 			(layer "F.SilkS")
 			(hide yes)
@@
 		)
 		(property "Value" "1N4007"
-			(at 0.1 1.475 360)
+			(at 0.1 1.475 0)
 			(layer "F.Fab")
 			(effects
@@
 		(tags "Diode")
 		(property "Reference" "D11"
-			(at 2.7 0 360)
+			(at 2.7 0 0)
 			(layer "F.SilkS")
 			(hide yes)
@@
 		)
 		(property "Value" "1N4007"
-			(at 0.1 1.475 360)
+			(at 0.1 1.475 0)
 			(layer "F.Fab")
 			(effects
@@
 		(tags "Diode")
 		(property "Reference" "D15"
-			(at 2.7 0 360)
+			(at 2.7 0 0)
 			(layer "F.SilkS")
 			(hide yes)
@@
 		)
 		(property "Value" "1N4007"
-			(at 0.1 1.475 360)
+			(at 0.1 1.475 0)
 			(layer "F.Fab")
 			(effects
@@
 		(tags "Diode")
 		(property "Reference" "D9"
-			(at 2.7 0 360)
+			(at 2.7 0 0)
 			(layer "F.SilkS")
 			(hide yes)
@@
 		)
 		(property "Value" "1N4007"
-			(at 0.1 1.475 360)
+			(at 0.1 1.475 0)
 			(layer "F.Fab")
 			(effects
@@
 		(tags "Diode")
 		(property "Reference" "D24"
-			(at 2.7 0 360)
+			(at 2.7 0 0)
 			(layer "F.SilkS")
 			(hide yes)
@@
 		)
 		(property "Value" "1N4007"
-			(at 0.1 1.475 360)
+			(at 0.1 1.475 0)
 			(layer "F.Fab")
 			(effects
@@
 		(tags "Diode")
 		(property "Reference" "D21"
-			(at 2.7 0 360)
+			(at 2.7 0 0)
 			(layer "F.SilkS")
 			(hide yes)
@@
 		)
 		(property "Value" "1N4007"
-			(at 0.1 1.475 360)
+			(at 0.1 1.475 0)
 			(layer "F.Fab")
 			(effects
@@
 		(tags "Diode")
 		(property "Reference" "D10"
-			(at 2.7 0 360)
+			(at 2.7 0 0)
 			(layer "F.SilkS")
 			(hide yes)
@@
 		)
 		(property "Value" "1N4007"
-			(at 0.1 1.475 360)
+			(at 0.1 1.475 0)
 			(layer "F.Fab")
 			(effects
@@
 		(at 67.075156 137.6925)
 		(property "Reference" "J13"
-			(at 17.78 -5.46 360)
+			(at 17.78 -5.46 0)
 			(layer "F.SilkS")
 			(effects
@@
 		)
 		(property "Value" "KF-5.08-8-V"
-			(at 17.78 5.11 360)
+			(at 17.78 5.11 0)
 			(layer "F.Fab")
 			(effects
@@
 		)
 		(fp_text user "${REFERENCE}"
-			(at 17.78 -5.46 360)
+			(at 17.78 -5.46 0)
 			(layer "F.Fab")
 			(effects
@@
 		(at 108.755156 137.6925)
 		(property "Reference" "J14"
-			(at 17.78 -5.46 360)
+			(at 17.78 -5.46 0)
 			(layer "F.SilkS")
 			(effects
@@
 		)
 		(property "Value" "KF-5.08-8-V"
-			(at 17.78 5.11 360)
+			(at 17.78 5.11 0)
 			(layer "F.Fab")
 			(effects
@@
 		)
 		(fp_text user "${REFERENCE}"
-			(at 17.78 -5.46 360)
+			(at 17.78 -5.46 0)
 			(layer "F.Fab")
 			(effects
@@
 		(at 150.435156 137.6925)
 		(property "Reference" "J15"
-			(at 17.78 -5.46 360)
+			(at 17.78 -5.46 0)
 			(layer "F.SilkS")
 			(effects
@@
 		)
 		(property "Value" "KF-5.08-8-V"
-			(at 17.78 5.11 360)
+			(at 17.78 5.11 0)
 			(layer "F.Fab")
 			(effects
@@
 		)
 		(fp_text user "${REFERENCE}"
-			(at 17.78 -5.46 360)
+			(at 17.78 -5.46 0)
 			(layer "F.Fab")
 			(effects
@@
 		(tags "Diode")
 		(property "Reference" "D13"
-			(at 2.7 0 360)
+			(at 2.7 0 0)
 			(layer "F.SilkS")
 			(hide yes)
@@
 		)
 		(property "Value" "1N4007"
-			(at 0.1 1.475 360)
+			(at 0.1 1.475 0)
 			(layer "F.Fab")
 			(effects
@@
 		(tags "Diode")
 		(property "Reference" "D19"
-			(at 2.7 0 360)
+			(at 2.7 0 0)
 			(layer "F.SilkS")
 			(hide yes)
@@
 		)
 		(property "Value" "1N4007"
-			(at 0.1 1.475 360)
+			(at 0.1 1.475 0)
 			(layer "F.Fab")
 			(effects
@@
 		)
 		(property "Field2" ""
-			(at 0 0 360)
+			(at 0 0 0)
 			(layer "F.Fab")
 			(hide yes)
@@
 		(tags "Diode")
 		(property "Reference" "D12"
-			(at 2.7 0 360)
+			(at 2.7 0 0)
 			(layer "F.SilkS")
 			(hide yes)
@@
 		)
 		(property "Value" "1N4007"
-			(at 0.1 1.475 360)
+			(at 0.1 1.475 0)
 			(layer "F.Fab")
 			(effects
@@
 		(tags "Diode")
 		(property "Reference" "D14"
-			(at 2.7 0 360)
+			(at 2.7 0 0)
 			(layer "F.SilkS")
 			(hide yes)
@@
 		)
 		(property "Value" "1N4007"
-			(at 0.1 1.475 360)
+			(at 0.1 1.475 0)
 			(layer "F.Fab")
 			(effects
@@
 		(tags "Diode")
 		(property "Reference" "D20"
-			(at 2.7 0 360)
+			(at 2.7 0 0)
 			(layer "F.SilkS")
 			(hide yes)
@@
 		)
 		(property "Value" "1N4007"
-			(at 0.1 1.475 360)
+			(at 0.1 1.475 0)
 			(layer "F.Fab")
 			(effects
@@
 		(tags "Diode")
 		(property "Reference" "D17"
-			(at 2.7 0 360)
+			(at 2.7 0 0)
 			(layer "F.SilkS")
 			(hide yes)
@@
 		)
 		(property "Value" "1N4007"
-			(at 0.1 1.475 360)
+			(at 0.1 1.475 0)
 			(layer "F.Fab")
 			(effects
@@
 		(tags "Diode")
 		(property "Reference" "D23"
-			(at 2.7 0 360)
+			(at 2.7 0 0)
 			(layer "F.SilkS")
 			(hide yes)
@@
 		)
 		(property "Value" "1N4007"
-			(at 0.1 1.475 360)
+			(at 0.1 1.475 0)
 			(layer "F.Fab")
 			(effects
@@
 	)
 	(segment
-		(start 236.9975 89.8975)
-		(end 247.3 100.2)
-		(width 1)
-		(layer "F.Cu")
-		(net 3)
-	)
-	(segment
-		(start 248.000156 100.900156)
-		(end 248.000156 131.9425)
-		(width 1)
-		(layer "F.Cu")
-		(net 3)
-	)
-	(segment
-		(start 216.243 89.8975)
-		(end 236.9975 89.8975)
-		(width 1)
+		(start 248.000156 97.800156)
+		(end 240.0975 89.8975)
+		(width 1.5)
 		(layer "F.Cu")
 		(net 3)
 	)
 	(segment
-		(start 247.3 100.2)
-		(end 247.605 100.505)
-		(width 1)
+		(start 248.000156 131.9425)
+		(end 248.000156 97.800156)
+		(width 1.5)
 		(layer "F.Cu")
 		(net 3)
 	)
 	(segment
-		(start 247.3 100.2)
-		(end 248.000156 100.900156)
-		(width 1)
+		(start 240.0975 89.8975)
+		(end 216.243 89.8975)
+		(width 1.5)
 		(layer "F.Cu")
 		(net 3)
@@
 	)
 	(segment
+		(start 243.935156 131.9575)
+		(end 243.950156 131.9425)
+		(width 1.5)
+		(layer "F.Cu")
+		(net 198)
+	)
+	(segment
+		(start 243.935156 138.2425)
+		(end 243.935156 131.9575)
+		(width 1.5)
+		(layer "F.Cu")
+		(net 198)
+	)
+	(segment
+		(start 233.435156 138.2425)
+		(end 233.435156 132.2175)
+		(width 1.5)
+		(layer "F.Cu")
+		(net 199)
+	)
+	(segment
+		(start 233.435156 132.2175)
+		(end 233.410156 132.1925)
+		(width 1.5)
+		(layer "F.Cu")
+		(net 199)
+	)
+	(segment

Commit message: feat <Wiring>: Complete wiring for power, RS485 and USB
Parts:
- moved LE10 32.0 mm to (140.4, 126.2)
- moved D16 32.0 mm to (142.2, 131.8)
- moved Q13 32.0 mm to (142.2, 129.0)
- moved R32 32.0 mm to (143.9, 126.2)
- moved R69 32.0 mm to (144.7, 128.7)
- moved R73 32.0 mm to (139.4, 128.8)
- moved R70 30.6 mm to (108.4, 128.7)
- moved D13 30.6 mm to (111.0, 131.8)
- moved LE7 30.6 mm to (109.1, 126.1)
- moved Q10 30.6 mm to (111.0, 128.9)
- moved R29 30.6 mm to (112.8, 126.1)
- moved R66 30.6 mm to (113.5, 128.6)
- moved U1 13.5 mm to (248.5, 79.6)
- moved C1 13.5 mm to (229.4, 43.5)
- moved C2 13.5 mm to (199.5, 89.9)
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Routing:
- net +24V: track 69.2 -> 444.2 mm
- net +3.3V: track 63.2 -> 376.7 mm, vias 0 -> 7
- net +3V3: track 23.2 -> 192.7 mm, vias 0 -> 2
- net +5V: track 112.1 -> 220.8 mm, vias 0 -> 1
- net /ConverterVoltTo4_20mA/DAC_4_20mA: track 5.62 -> 112.2 mm, vias 0 -> 2
- net /ESP32/BOOT: track 18.7 -> 117.5 mm, vias 0 -> 2
- net /RS485/RS485_input.RX: track 0.00 -> 61.6 mm
- net /STM32/USB_Detect: track 1.90 -> 63.5 mm, vias 0 -> 2
- net /RS485/RS485_input.TX: track 0.00 -> 60.8 mm
- net /RS485/RS485_input.DERE: track 4.58 -> 64.8 mm, vias 0 -> 2
- net /STM32/USB_DM: track 16.1 -> 69.5 mm, vias 1 -> 2
- net /STM32/USB_DP: track 26.9 -> 79.2 mm, vias 3 -> 4
- net /VBUS: track 15.4 -> 46.4 mm, vias 0 -> 2
- net /LORA/RA02.MOSI: track 23.3 -> 47.7 mm, vias 0 -> 1
- net GND: track 142.1 -> 119.6 mm, vias 0 -> 1
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
Commit message: fix board edge cut
Routing:
- net (no net): track 433.1 -> 0.00 mm
Other:
- board size 254 x 135 mm -> 252.8 x 129 mm
Changed lines of the file:
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@@
 	)
 	(gr_line
-		(start 23.900371 26)
-		(end 23.900371 145)
-		(locked yes)
-		(stroke
-			(width 0.2)
-			(type default)
-		)
-		(layer "Edge.Cuts")
-	)
-	(gr_arc
-		(start 268.900371 17)
-		(mid 275.264351 19.636029)
-		(end 277.900371 26)
-		(locked yes)
+		(start 263 17)
+		(end 36.192388 17)
 		(stroke
 			(width 0.05)
@@
 	)
 	(gr_arc
-		(start 277.9 143.136039)
-		(mid 275.295501 149.492344)
-		(end 268.900371 152)
-		(locked yes)
+		(start 23.192388 30)
+		(mid 27 20.807612)
+		(end 36.192388 17)
 		(stroke
-			(width 0.2)
+			(width 0.05)
 			(type default)
 		)
@@
 	)
 	(gr_arc
-		(start 23.900371 26)
-		(mid 26.536408 19.636029)
-		(end 32.900371 17)
-		(locked yes)
+		(start 36.192388 146)
+		(mid 27 142.192388)
+		(end 23.192388 133)
 		(stroke
 			(width 0.05)
@@
 	)
 	(gr_line
-		(start 268.900371 17)
-		(end 32.900371 17)
-		(locked yes)
+		(start 276 30)
+		(end 276 133)
 		(stroke
 			(width 0.05)
@@
 	)
 	(gr_line
-		(start 30.9 152)
-		(end 268.900371 152)
-		(locked yes)
+		(start 36.192388 146)
+		(end 263 146)
 		(stroke
-			(width 0.2)
+			(width 0.05)
+			(type default)
+		)
+		(layer "Edge.Cuts")
+	)
+	(gr_arc
+		(start 276 133)
+		(mid 272.192388 142.192388)
+		(end 263 146)
+		(stroke
+			(width 0.05)
 			(type default)
 		)
@@
 	)
 	(gr_line
-		(start 277.900371 143.5)
-		(end 277.900371 26)
-		(locked yes)
+		(start 23.192388 30)
+		(end 23.192388 133)
 		(stroke
-			(width 0.2)
+			(width 0.05)
 			(type default)
 		)
@@
 	)
 	(gr_arc
-		(start 30.921631 151.999501)
-		(mid 25.940739 149.997522)
-		(end 23.903154 145.031108)
-		(locked yes)
+		(start 263 17)
+		(mid 272.192388 20.807612)
+		(end 276 30)
 		(stroke
-			(width 0.2)
+			(width 0.05)
 			(type default)
 		)
@@
 		)
 	)
-	(dimension
-		(type aligned)
-		(layer "F.Cu")
-		(pts
-			(xy 270.9 47) (xy 270.9 122)
-		)
-		(height -9)
-		(gr_text "2952.7559 mils"
-			(at 278.1 84.5 90)
-			(layer "F.Cu")
-			(effects
-				(font
-					(size 1.5 1.5)
-					(thickness 0.3)
-				)
-			)
-		)
-		(format
-			(prefix "")
-			(suffix "")
-			(units 3)
-			(units_format 1)
-			(precision 4)
-		)
-		(style
-			(thickness 0.2)
-			(arrow_length 1.27)
-			(text_position_mode 0)
-			(extension_height 0.58642)
-			(extension_offset 0.5) keep_text_aligned)
-	)
-	(dimension
-		(type aligned)
-		(layer "F.Cu")
-		(pts
-			(xy 30.9 122) (xy 30.9 152)
-		)
-		(height 9.199999)
-		(gr_text "1181.1024 mils"
-			(at 19.900001 137 90)
-			(layer "F.Cu")
-			(effects
-				(font
-					(size 1.5 1.5)
-					(thickness 0.3)
-				)
-			)
-		)
-		(format
-			(prefix "")
-			(suffix "")
-			(units 3)
-			(units_format 1)
-			(precision 4)
-		)
-		(style
-			(thickness 0.2)
-			(arrow_length 1.27)
-			(text_position_mode 0)
-			(extension_height 0.58642)
-			(extension_offset 0.5) keep_text_aligned)
-	)
-	(dimension
-		(type aligned)
-		(layer "F.Cu")
-		(pts
-			(xy 30.9 47) (xy 30.9 122)
-		)
-		(height 9.2)
-		(gr_text "2952.7559 mils"
-			(at 19.9 84.5 90)
-			(layer "F.Cu")
-			(effects
-				(font
-					(size 1.5 1.5)
-					(thickness 0.3)
-				)
-			)
-		)
-		(format
-			(prefix "")
-			(suffix "")
-			(units 3)
-			(units_format 1)
-			(precision 4)
-		)
-		(style
-			(thickness 0.2)
-			(arrow_length 1.27)
-			(text_position_mode 0)
-			(extension_height 0.58642)
-			(extension_offset 0.5) keep_text_aligned)
-	)
 	(segment
-		(start 278.527876 22.011934)
-		(end 268.615942 12.1)
-		(width 0.25)
-		(layer "F.Cu")
-		(net 0)
-	)
-	(segment
-		(start 290.2 55)
-		(end 290.2 135.471876)
-		(width 0.25)
-		(layer "F.Cu")
-		(net 0)
-	)
-	(segment
-		(start 290.2 135.471876)
-		(end 278.527876 147.144)
-		(width 0.25)
-		(layer "F.Cu")
-		(net 0)
-	)
-	(segment
-		(start 86.6 12.1)
-		(end 82.325 16.375)
-		(width 0.25)
-		(layer "F.Cu")
-		(net 0)
-	)
-	(segment
-		(start 82.325 16.375)
-		(end 73.425 16.375)
-		(width 0.25)
-		(layer "F.Cu")
-		(net 0)
-	)
-	(segment
-		(start 278.527876 147.144)
-		(end 278.527876 22.011934)
-		(width 0.25)
-		(layer "F.Cu")
-		(net 0)
-	)
-	(segment
-		(start 268.615942 12.1)
-		(end 86.6 12.1)
-		(width 0.25)
-		(layer "F.Cu")
-		(net 0)
-	)
-	(segment

Commit message: layout p1
Parts:
- removed J7: Conn_02x03_Odd_Even, Connector_PinHeader_2.54mm:PinHeader_2x03_P2.54mm_Vertical
- R53: value 5k1 -> 1k5
- moved C20 84.7 mm to (66.6, 79.6)
- moved R22 84.7 mm to (65.9, 74.5)
- moved U5 84.7 mm to (69.6, 74.5)
- moved Y2 84.7 mm to (68.2, 84.8)
- moved C21 84.7 mm to (69.9, 79.6)
- moved C22 84.7 mm to (64.0, 72.4)
- moved D8 84.7 mm to (63.3, 76.3)
- moved R23 84.7 mm to (62.3, 72.4)
- moved R24 84.4 mm to (66.8, 70.1)
- moved R19 84.3 mm to (79.7, 35.9), turned to 0 degrees
- moved C18 74.0 mm to (83.1, 22.7), turned to 90 degrees
- moved SW2 70.8 mm to (85.9, 24.4), turned to 90 degrees
- moved R20 69.2 mm to (83.1, 26.1), turned to 90 degrees
- moved RV2 43.3 mm to (87.6, 72.1), turned to 180 degrees
- moved R118 39.7 mm to (84.1, 72.1), turned to -90 degrees
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Connections:
- C40 pad 1: +3V3 -> +3.3V
- D8 pad 1: +3V3 -> +3.3V
- FL1 pad 1: /DualPowerSupply-220V-to-24V_5V_AM22/220V_N -> Net-(C1-Pad2)
- FL1 pad 3: Net-(C1-Pad2) -> /DualPowerSupply-220V-to-24V_5V_AM22/220V_N
- J10 pad 6: +3V3 -> +3.3V
- J11 pad 13: +3V3 -> +3.3V
- J13 pad 4: /16ValveDriver/4ValveDriveOutput/VAN3- -> /16ValveDriver/4ValveDriveOutput/VAN2-
- J13 pad 6: /16ValveDriver/4ValveDriveOutput/VAN2- -> /16ValveDriver/4ValveDriveOutput/VAN3-
- J14 pad 4: /16ValveDriver/4ValveDriveOutput1/VAN3- -> /16ValveDriver/4ValveDriveOutput1/VAN2-
- J14 pad 6: /16ValveDriver/4ValveDriveOutput1/VAN2- -> /16ValveDriver/4ValveDriveOutput1/VAN3-
- J15 pad 4: /16ValveDriver/4ValveDriveOutput2/VAN3- -> /16ValveDriver/4ValveDriveOutput2/VAN2-
- J15 pad 6: /16ValveDriver/4ValveDriveOutput2/VAN2- -> /16ValveDriver/4ValveDriveOutput2/VAN3-
- J16 pad 4: /16ValveDriver/4ValveDriveOutput3/VAN3- -> /16ValveDriver/4ValveDriveOutput3/VAN2-
- J16 pad 6: /16ValveDriver/4ValveDriveOutput3/VAN2- -> /16ValveDriver/4ValveDriveOutput3/VAN3-
- J9 pad 6: +3V3 -> +3.3V
- JP1 pad 1: +3V3 -> +3.3V
- Q1 pad 1: +3V3 -> +3.3V
- Q2 pad 1: +3V3 -> +3.3V
- Q3 pad 1: +3V3 -> +3.3V
- Q4 pad 1: +3V3 -> +3.3V
- Q5 pad 1: +3V3 -> +3.3V
- R118 pad 1: +3V3 -> +3.3V
- R14 pad 1: /STM32/BOOT1 -> GND
- R15 pad 1: /STM32/BOOT0 -> GND
- R15 pad 2: Net-(U3-BOOT0) -> /STM32/BOOT0
- R20 pad 1: +3V3 -> +3.3V
- R21 pad 1: +3V3 -> +3.3V
- R41 pad 1: +3V3 -> +3.3V
- R42 pad 1: +3V3 -> +3.3V
- R43 pad 1: +3V3 -> +3.3V
- R44 pad 1: +3V3 -> +3.3V
- R45 pad 1: +3V3 -> +3.3V
- RV2 pad 3: +3V3 -> +3.3V
- U21 pad 8: +3V3 -> +3.3V
- U3 pad 44: Net-(U3-BOOT0) -> /STM32/BOOT0
Routing:
- net +3V3: track 192.7 -> 0.00 mm, vias 2 -> 0
- net +24V: track 444.2 -> 322.3 mm
- net /ESP32/BOOT: track 117.5 -> 0.00 mm, vias 2 -> 0
- net +3.3V: track 376.7 -> 492.0 mm, vias 7 -> 14
- net +5V: track 220.8 -> 318.8 mm, vias 1 -> 3
- net /ConverterVoltTo4_20mA/DAC_4_20mA: track 112.2 -> 43.5 mm
- net /RS485/RS485_input.RX: track 61.6 -> 2.27 mm
- net /RS485/RS485_input.TX: track 60.8 -> 2.26 mm
- net /RS485/RS485_input.DERE: track 64.8 -> 6.66 mm
- net GND: track 119.6 -> 173.7 mm, vias 1 -> 70
- net /16ValveDriver/ValveDriver1: track 3.33 -> 47.8 mm
- net /16ValveDriver/OpAmpOutput1: track 1.96 -> 43.6 mm, vias 0 -> 2
- net Net-(Q6-S): track 1.81 -> 36.9 mm, vias 0 -> 2
- net /16ValveDriver/ValveDriver8: track 3.28 -> 37.3 mm
- net /16ValveDriver/OpAmpOutput4: track 1.96 -> 32.8 mm, vias 0 -> 2
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- added copper zone on F.Cu, net +3.3V
- added copper zone on B.Cu, net /VBUS
- added copper zone on F.Cu, net /VBUS
- added copper zone on B.Cu, net GND
- added copper zone on F.Cu, net GND
Other:
- board size 252.8 x 129 mm -> 252.8 x 135 mm

Commit message: Layout p2, fix Analog VCC and GND for opamp circuit
Parts:
- moved R24 38.8 mm to (99.2, 91.4), turned to -90 degrees
- moved C40 38.1 mm to (68.3, 104.7)
- moved R118 38.1 mm to (73.3, 108.7)
- moved R119 38.1 mm to (68.3, 112.2)
- moved RV2 38.1 mm to (76.8, 108.7)
- moved U21 38.1 mm to (68.3, 108.4)
- moved R23 37.5 mm to (96.9, 86.9), turned to 0 degrees
- moved C22 36.7 mm to (96.9, 88.7), turned to 180 degrees
- moved R22 33.0 mm to (94.8, 90.5), turned to 180 degrees
- moved U5 32.0 mm to (94.8, 94.2), turned to 0 degrees
- moved D8 31.8 mm to (92.9, 87.9), turned to -90 degrees
- moved C20 25.9 mm to (89.7, 91.2), turned to 90 degrees
- moved C21 24.8 mm to (89.7, 94.5), turned to -90 degrees
- moved Y2 18.1 mm to (84.5, 92.8), turned to 180 degrees
- moved C38 12.7 mm to (42.5, 64.2)
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Connections:
- net /STM32/PC14 renamed /PCF8563/CLKOUT
- net Net-(U15-Q7) renamed /ReadValveState/74HC165_CascadeDATA
- C32 pad 1: +5V -> /16ValveDriver/AnalogVCC
- C32 pad 2: GND -> GNDA
- C33 pad 1: +5V -> /16ValveDriver/AnalogVCC
- C33 pad 2: GND -> GNDA
- C34 pad 1: +5V -> /16ValveDriver/AnalogVCC
- C34 pad 2: GND -> GNDA
- C35 pad 1: +5V -> /16ValveDriver/AnalogVCC
- C35 pad 2: GND -> GNDA
- C40 pad 1: +3.3V -> +5V
- D25 pad 3: /LORA/RA02.MOSI -> /SDcard/DetectCard
- D25 pad 4: /SDcard/SDcardSPI.CLK -> /LORA/RA02.MISO
- D25 pad 5: /LORA/RA02.MOSI -> /LORA/RA02.SCK
- D25 pad 6: /SDcard/DetectCard -> /LORA/RA02.MOSI
- J17 pad 5: /SDcard/SDcardSPI.CLK -> /LORA/RA02.SCK
- J17 pad 7: /LORA/RA02.MOSI -> /LORA/RA02.MISO
- Q18 pad 1: /16ValveDriver/ValveDriver13 -> /16ValveDriver/4ValveDriveOutput3/ValveInput1
- Q19 pad 1: /16ValveDriver/ValveDriver14 -> /16ValveDriver/4ValveDriveOutput3/ValveInput2
- Q20 pad 1: /16ValveDriver/ValveDriver15 -> /16ValveDriver/4ValveDriveOutput3/ValveInput3
- Q21 pad 1: /16ValveDriver/ValveDriver16 -> /16ValveDriver/4ValveDriveOutput3/ValveInput4
- R100 pad 1: +5V -> /16ValveDriver/AnalogVCC
- R101 pad 1: +5V -> /16ValveDriver/AnalogVCC
- R118 pad 1: +3.3V -> +5V
- R118 pad 2: /VoltageReference/MCP41010/AnalogVCC -> /16ValveDriver/AnalogVCC
- R119 pad 2: /VoltageReference/MCP41010/AnalogGND -> GNDA
- R54 pad 2: GND -> GNDA
- R55 pad 2: GND -> GNDA
- R56 pad 2: GND -> GNDA
- R57 pad 2: GND -> GNDA
- R58 pad 2: GND -> GNDA
- R59 pad 2: GND -> GNDA
- R60 pad 2: GND -> GNDA
- R61 pad 2: GND -> GNDA
- R62 pad 1: +5V -> /16ValveDriver/AnalogVCC
- R63 pad 1: +5V -> /16ValveDriver/AnalogVCC
- R64 pad 1: +5V -> /16ValveDriver/AnalogVCC
- R65 pad 1: +5V -> /16ValveDriver/AnalogVCC
- R66 pad 2: GND -> GNDA
- R67 pad 2: GND -> GNDA
- R68 pad 2: GND -> GNDA
- R69 pad 2: GND -> GNDA
- R70 pad 2: GND -> GNDA
- R71 pad 2: GND -> GNDA
- R72 pad 2: GND -> GNDA
- R73 pad 2: GND -> GNDA
- R74 pad 1: +5V -> /16ValveDriver/AnalogVCC
- R75 pad 1: +5V -> /16ValveDriver/AnalogVCC
- R76 pad 1: +5V -> /16ValveDriver/AnalogVCC
- R77 pad 1: +5V -> /16ValveDriver/AnalogVCC
- R78 pad 2: GND -> GNDA
- R79 pad 2: GND -> GNDA
- R80 pad 2: GND -> GNDA
- R81 pad 2: GND -> GNDA
- R82 pad 2: GND -> GNDA
- R83 pad 2: GND -> GNDA
- R84 pad 2: GND -> GNDA
- R85 pad 2: GND -> GNDA
- R86 pad 1: +5V -> /16ValveDriver/AnalogVCC
- R87 pad 1: +5V -> /16ValveDriver/AnalogVCC
- R88 pad 1: +5V -> /16ValveDriver/AnalogVCC
- R89 pad 1: +5V -> /16ValveDriver/AnalogVCC
- R90 pad 1: /16ValveDriver/ValveDriver13 -> /16ValveDriver/4ValveDriveOutput3/ValveInput1
- R90 pad 2: GND -> GNDA
- R91 pad 1: /16ValveDriver/ValveDriver14 -> /16ValveDriver/4ValveDriveOutput3/ValveInput2
- R91 pad 2: GND -> GNDA
- R92 pad 1: /16ValveDriver/ValveDriver15 -> /16ValveDriver/4ValveDriveOutput3/ValveInput3
- R92 pad 2: GND -> GNDA
- R93 pad 1: /16ValveDriver/ValveDriver16 -> /16ValveDriver/4ValveDriveOutput3/ValveInput4
- R93 pad 2: GND -> GNDA
- R94 pad 2: GND -> GNDA
- R95 pad 2: GND -> GNDA
- R96 pad 2: GND -> GNDA
- R97 pad 2: GND -> GNDA
- R98 pad 1: +5V -> /16ValveDriver/AnalogVCC
- R99 pad 1: +5V -> /16ValveDriver/AnalogVCC
- U11 pad 11: GND -> GNDA
- U11 pad 4: +5V -> /16ValveDriver/AnalogVCC
- U12 pad 11: GND -> GNDA
- U12 pad 4: +5V -> /16ValveDriver/AnalogVCC
- U13 pad 11: GND -> GNDA
- U13 pad 4: +5V -> /16ValveDriver/AnalogVCC
- U14 pad 11: GND -> GNDA
- U14 pad 4: +5V -> /16ValveDriver/AnalogVCC
- U21 pad 5: /VoltageReference/MCP41010/AnalogVCC -> /16ValveDriver/AnalogVCC
- U21 pad 7: /VoltageReference/MCP41010/AnalogGND -> GNDA
- U21 pad 8: +3.3V -> +5V
Routing:
- net +5V: track 318.8 -> 582.4 mm, vias 3 -> 28
- net /LORA/RA02.SCK: track 0.00 -> 192.9 mm, vias 0 -> 6
- net /LORA/RA02.CS_LORA: track 0.00 -> 171.6 mm, vias 0 -> 4
- net /LORA/RA02.MISO: track 0.00 -> 168.2 mm, vias 0 -> 6
- net /LORA/RA02.MOSI: track 40.4 -> 191.0 mm, vias 0 -> 6
- net /LORA/LoRaReceivedInterrupt: track 0.00 -> 144.3 mm, vias 0 -> 2
- net +3.3V: track 492.0 -> 634.1 mm, vias 14 -> 33
- net /AMS5915/i2c.SCL: track 6.70 -> 147.8 mm, vias 2 -> 4
- net /STM32/595.SRCLK: track 0.00 -> 133.8 mm, vias 0 -> 6
- net /STM32/595.RCLK: track 0.00 -> 132.7 mm, vias 0 -> 6
- net /AMS5915/i2c.SDA: track 8.13 -> 135.9 mm, vias 2 -> 4
- net /ESP32/TX_ESP32: track 13.8 -> 141.4 mm, vias 1 -> 4
- net /SDcard/DetectCard: track 10.7 -> 136.1 mm, vias 0 -> 2
- net /ReadValveState/OE: track 0.00 -> 122.7 mm, vias 0 -> 6
- net /ESP32/RX_ESP32: track 0.00 -> 122.0 mm, vias 0 -> 4
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- added copper zone on B.Cu, net +3.3V
- added copper zone on B.Cu, net +5V
- added copper zone on B.Cu, net GNDA
- added copper zone on F.Cu, net GNDA
