File: DongTamV2.kicad_pcb (KiCad board)
At the start: 2 copper layers, 252.8 x 135 mm, 287 parts, among them J1 KF128, J10 Conn_01x05_Male, J11 IDC_02x07, J12 USB_C_Receptacle, J13 KF-5.08-8-V, J14 KF-5.08-8-V, J15 KF-5.08-8-V, J16 KF-5.08-8-V, J17 Micro_SD_Card_Det1, J18 HT3.96mm-3P, J2 KF128, J3 KF128, J4 KF128, J5 KF128, J6 Conn_01x02_Male, J9 Conn_01x05_Male, Q1 SI2302/BSS138, Q10 SI2302, Q11 SI2302, Q12 SI2302, Q13 SI2302, Q14 SI2302, Q15 SI2302, Q16 SI2302, Q17 SI2302, Q18 SI2302, Q19 SI2302, Q2 SI2302/BSS138, Q20 SI2302, Q21 SI2302, Q22 MMBT3904, Q3 SI2302/BSS138, Q4 SI2302/BSS138, Q5 SI2302/BSS138, Q6 SI2302, Q7 SI2302, Q8 SI2302, Q9 SI2302, SW1 PTS810, SW2 PTS810, SW3 PTS810, U1 AM22-24W2405V, U10 LD1117, U11 LM324, U12 LM324, U13 LM324, U14 LM324, U15 74HC165, U16 74HC165, U17 RF_Module_Ai-Thinker-Ra-02, U18 LM324, U19 LM317_TO-252, U2 SP3485EN, U20 TL431, U21 MCP41010, U3 MCU_STM32F103C8Tx, U4 ESP32-WROOM-32, U5 PCF8563TS, U6 AMS5915, U7 74HC595, U8 74HC595, U9 USBLC6-2SC6, Y1 16MHz, Y2 MC-306

Commit message: Complete layout, HW685 not layout yet
Parts:
- moved R98 13.4 mm to (203.0, 120.0), turned to 180 degrees
- moved R101 13.3 mm to (207.2, 120.0), turned to 0 degrees
- moved C34 11.9 mm to (156.2, 114.3), turned to 180 degrees
- moved C33 10.8 mm to (123.3, 115.1), turned to -90 degrees
- moved D15 10.8 mm to (132.3, 131.8)
- moved LE9 10.8 mm to (130.3, 126.0)
- moved Q12 10.8 mm to (132.3, 129.0)
- moved R31 10.8 mm to (134.0, 126.0)
- moved R68 10.8 mm to (134.8, 128.7)
- moved R72 10.8 mm to (129.4, 128.8)
- moved R100 10.5 mm to (207.2, 108.7), turned to 0 degrees
- moved R99 10.5 mm to (203.1, 108.7), turned to 180 degrees
- moved LE8 9.89 mm to (119.8, 126.1)
- moved D14 9.89 mm to (121.7, 131.8)
- moved Q11 9.89 mm to (121.7, 129.1)
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Connections:
- Q18 pad 1: /16ValveDriver/4ValveDriveOutput3/ValveInput1 -> /16ValveDriver/ValveDriver13
- Q19 pad 1: /16ValveDriver/4ValveDriveOutput3/ValveInput2 -> /16ValveDriver/ValveDriver14
- Q20 pad 1: /16ValveDriver/4ValveDriveOutput3/ValveInput3 -> /16ValveDriver/ValveDriver15
- Q21 pad 1: /16ValveDriver/4ValveDriveOutput3/ValveInput4 -> /16ValveDriver/ValveDriver16
- R54 pad 2: GNDA -> GND
- R55 pad 2: GNDA -> GND
- R56 pad 2: GNDA -> GND
- R57 pad 2: GNDA -> GND
- R58 pad 2: GNDA -> GND
- R59 pad 2: GNDA -> GND
- R60 pad 2: GNDA -> GND
- R61 pad 2: GNDA -> GND
- R66 pad 2: GNDA -> GND
- R67 pad 2: GNDA -> GND
- R68 pad 2: GNDA -> GND
- R69 pad 2: GNDA -> GND
- R70 pad 2: GNDA -> GND
- R71 pad 2: GNDA -> GND
- R72 pad 2: GNDA -> GND
- R73 pad 2: GNDA -> GND
- R78 pad 2: GNDA -> GND
- R79 pad 2: GNDA -> GND
- R80 pad 2: GNDA -> GND
- R81 pad 2: GNDA -> GND
- R82 pad 2: GNDA -> GND
- R83 pad 2: GNDA -> GND
- R84 pad 2: GNDA -> GND
- R85 pad 2: GNDA -> GND
- R90 pad 1: /16ValveDriver/4ValveDriveOutput3/ValveInput1 -> /16ValveDriver/ValveDriver13
- R90 pad 2: GNDA -> GND
- R91 pad 1: /16ValveDriver/4ValveDriveOutput3/ValveInput2 -> /16ValveDriver/ValveDriver14
- R91 pad 2: GNDA -> GND
- R92 pad 1: /16ValveDriver/4ValveDriveOutput3/ValveInput3 -> /16ValveDriver/ValveDriver15
- R92 pad 2: GNDA -> GND
- R93 pad 1: /16ValveDriver/4ValveDriveOutput3/ValveInput4 -> /16ValveDriver/ValveDriver16
- R93 pad 2: GNDA -> GND
- R94 pad 2: GNDA -> GND
- R95 pad 2: GNDA -> GND
- R96 pad 2: GNDA -> GND
- R97 pad 2: GNDA -> GND
- RV2 pad 1: GND -> GNDA
- RV2 pad 3: +3.3V -> /16ValveDriver/AnalogVCC
Routing:
- net GND: track 241.7 -> 721.6 mm, vias 97 -> 186
- net /16ValveDriver/AnalogVCC: track 52.5 -> 277.5 mm, vias 2 -> 20
- net /16ValveDriver/REF: track 26.3 -> 184.9 mm, vias 0 -> 6
- net /STM32/4_20mA: track 0.00 -> 69.6 mm
- net +5V: track 582.4 -> 645.5 mm, vias 28 -> 39
- net /16ValveDriver/OpAmpOutput9: track 0.00 -> 50.8 mm, vias 0 -> 2
- net /16ValveDriver/OpAmpOutput16: track 0.00 -> 45.4 mm, vias 0 -> 2
- net /16ValveDriver/OpAmpOutput10: track 0.00 -> 36.3 mm, vias 0 -> 2
- net Net-(Q10-S): track 1.70 -> 34.9 mm, vias 0 -> 4
- net /16ValveDriver/OpAmpOutput15: track 0.00 -> 32.8 mm, vias 0 -> 2
- net /16ValveDriver/OpAmpOutput12: track 0.00 -> 32.0 mm, vias 0 -> 2
- net /16ValveDriver/OpAmpOutput13: track 0.00 -> 29.9 mm, vias 0 -> 2
- net Net-(Q21-S): track 1.80 -> 31.3 mm, vias 0 -> 2
- net Net-(Q17-S): track 1.67 -> 28.8 mm, vias 0 -> 2
- net /STM32/RX_LOG: track 0.00 -> 26.3 mm, vias 0 -> 1
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