File: DongTamV2.kicad_pcb (KiCad board)
At the start: 2 copper layers, 252.8 x 135 mm, 287 parts, among them J1 KF128, J10 Conn_01x05_Male, J11 IDC_02x07, J12 USB_C_Receptacle, J13 KF-5.08-8-V, J14 KF-5.08-8-V, J15 KF-5.08-8-V, J16 KF-5.08-8-V, J17 Micro_SD_Card_Det1, J18 HT3.96mm-3P, J2 KF128, J3 KF128, J4 KF128, J5 KF128, J6 Conn_01x02_Male, J9 Conn_01x05_Male, Q1 SI2302/BSS138, Q10 SI2302, Q11 SI2302, Q12 SI2302, Q13 SI2302, Q14 SI2302, Q15 SI2302, Q16 SI2302, Q17 SI2302, Q18 SI2302, Q19 SI2302, Q2 SI2302/BSS138, Q20 SI2302, Q21 SI2302, Q22 MMBT3904, Q3 SI2302/BSS138, Q4 SI2302/BSS138, Q5 SI2302/BSS138, Q6 SI2302, Q7 SI2302, Q8 SI2302, Q9 SI2302, SW1 PTS810, SW2 PTS810, SW3 PTS810, U1 AM22-24W2405V, U10 LD1117, U11 LM324, U12 LM324, U13 LM324, U14 LM324, U15 74HC165, U16 74HC165, U17 RF_Module_Ai-Thinker-Ra-02, U18 LM324, U19 LM317_TO-252, U2 SP3485EN, U20 TL431, U21 MCP41010, U3 MCU_STM32F103C8Tx, U4 ESP32-WROOM-32, U5 PCF8563TS, U6 AMS5915, U7 74HC595, U8 74HC595, U9 USBLC6-2SC6, Y1 16MHz, Y2 MC-306

Commit message: feat: adding HW685 module
Parts:
- added G***: LOGO, LOGO, F.Cu at (74.5, 76.0)
- added J7: Conn_01x03_Pin, Connector_PinHeader_2.54mm:PinHeader_1x03_P2.54mm_Vertical, F.Cu at (56.7, 112.7)
- added JP2: SolderJumper_2_Open, SpiritBoi_Footprint_Library:SolderJumper-2_P1.3mm_Open_TrianglePad1.0x1.5mm, F.Cu at (55.7, 122.2)
- added U22: L7815, SpiritBoi_Footprint_Library:Package-IC-Vert-SMD-TO_263-2_TabPin2, F.Cu at (45.5, 136.1)
- added U23: L7812, SpiritBoi_Footprint_Library:Package-IC-Vert-SMD-TO_263-2_TabPin2, F.Cu at (45.5, 111.2)
- D10, D11, D12, D13, D14, D15, D16, D17, D18, D19, D20, D21, D22, D23, D24, D9: value 1N4007 -> 1N4148W
- moved R116 4.49 mm to (133.6, 42.3)
- moved R113 4.48 mm to (135.7, 42.2)
- moved REF** 4.38 mm to (119.8, 20.5)
- moved D25 1.95 mm to (42.7, 69.0)
- moved J17 1.32 mm to (27.2, 69.0)
- moved R63 0.26 mm to (88.4, 108.4)
- moved D9 0.17 mm to (68.5, 131.9)
Connections:
- U3 pad 19: /STM32/4_20mA -> /HW685/4-20mA
Routing:
- net /HW685/4-20mA: track 0.00 -> 140.7 mm, vias 0 -> 1
- net /STM32/4_20mA: track 69.6 -> 0.00 mm
- net +24V: track 431.5 -> 466.9 mm
- net +15V: track 0.00 -> 23.1 mm
- net GND: track 721.6 -> 726.7 mm, vias 186 -> 188
- net Net-(Q22-E): track 3.75 -> 8.74 mm
- net Net-(U18C--): track 15.7 -> 10.8 mm
- net +5V: track 645.5 -> 647.7 mm
- net /LORA/RA02.MISO: track 168.2 -> 166.5 mm
- net Net-(R114-Pad2): track 11.8 -> 13.3 mm, vias 0 -> 2
- net /16ValveDriver/AnalogVCC: track 277.5 -> 276.0 mm
- net +3.3V: track 636.0 -> 637.3 mm
- net Net-(U18A--): track 13.7 -> 15.0 mm
- net /LORA/RA02.SCK: track 191.7 -> 190.5 mm
- net /LORA/RA02.CS_LORA: track 171.6 -> 172.7 mm
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- added copper zone on F.Cu, net +12V
Other:
- board text added: "220V~"
- board text added: "24V"
- board text added: "5V"
- board text added: "A"
- board text added: "ESP BOOT"
- board text added: "ESP RESET"
- board text added: "Earth B"
- board text added: "GND"
- board text added: "GND RST TX RX BOOT 3.3V"
- board text added: "GND TDI TDO TCK TMS 3.3V"
- board text added: "HW685"
- board text added: "Made by Trương Minh Khoa"
- board text added: "OUT"
- board text added: "RS485"
- board text added: "RX SWCLK TX SWDIO GND GND 5V 3.3V"
- board text added: "ST RST"
- board text added: "VAN1"
- board text added: "VAN10"
- board text added: "VAN11"
- board text added: "VAN12"
- board text added: "VAN13"
- board text added: "VAN14"
- board text added: "VAN15"
- board text added: "VAN16"
- board text added: "VAN2"
- board text added: "VAN3"
- board text added: "VAN4"
- board text added: "VAN5"
- board text added: "VAN6"
- board text added: "VAN7"
- board text added: "VAN8"
- board text added: "VAN9"
- board text added: "bypass 15V"
- board text added: "spirit boi"
- board text added: "Đồng Tâm V2.1"
- board text removed: "Còn mạch đọc 4-20mA"
