File: ValveDriveOutput.kicad_sch (KiCad schematic)
At the start: 23 parts, among them J14 Screw_Terminal_01x08, Q6 SI2302, Q7 SI2302, Q8 SI2302, Q9 SI2302, U11 LM324

Commit message: finish some unconnect pins, draw edge cut board
Parts:
- J14: value Screw_Terminal_01x08 -> KF-5.08-8-V
Changed lines of the file:
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@@
 			)
 		)
-		(property "Value" "Screw_Terminal_01x08"
+		(property "Value" "KF-5.08-8-V"
 			(at 187.96 72.39 0)
 			(effects

Commit message: Add LORA, SDcard and Volt to 4_20mA scheamtic
Parts:
- J13: renamed from J14; footprint TerminalBlock:TerminalBlock_bornier-8_P5.08mm -> SpiritBoi_Footprint_Library:TerminalBlock-Horz-THT-8P-P5.08mm-KF2EDG_Pluggable
- renumbered D8 to D10, D9 to D11, D10 to D12, D7 to D9
Changed lines of the file:
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@@
 		(on_board yes)
 		(dnp no)
-		(property "Reference" "D9"
+		(property "Reference" "D11"
 			(at 74.93 114.2999 90)
 			(effects
@@
 			(project "DongTamV2"
 				(path "/2303d546-b88a-4ab0-aee1-26e3b32ac9d7/2c066284-8887-41f4-b61e-b40cb8a906fb/0f07157a-883c-4ea4-935e-e968b282f133"
-					(reference "D9")
-					(unit 1)
-				)
-				(path "/2303d546-b88a-4ab0-aee1-26e3b32ac9d7/2c066284-8887-41f4-b61e-b40cb8a906fb/64421711-110b-460c-9945-866904db2698"
-					(reference "D13")
-					(unit 1)
-				)
-				(path "/2303d546-b88a-4ab0-aee1-26e3b32ac9d7/2c066284-8887-41f4-b61e-b40cb8a906fb/2f9aecb0-00e3-4033-a162-064bbf4c14dd"
-					(reference "D17")
-					(unit 1)
-				)
-				(path "/2303d546-b88a-4ab0-aee1-26e3b32ac9d7/2c066284-8887-41f4-b61e-b40cb8a906fb/77ab04e0-ca17-45de-8f43-d4b5585142b1"
-					(reference "D21")
+					(reference "D11")
+					(unit 1)
+				)
+				(path "/2303d546-b88a-4ab0-aee1-26e3b32ac9d7/2c066284-8887-41f4-b61e-b40cb8a906fb/64421711-110b-460c-9945-866904db2698"
+					(reference "D15")
+					(unit 1)
+				)
+				(path "/2303d546-b88a-4ab0-aee1-26e3b32ac9d7/2c066284-8887-41f4-b61e-b40cb8a906fb/2f9aecb0-00e3-4033-a162-064bbf4c14dd"
+					(reference "D19")
+					(unit 1)
+				)
+				(path "/2303d546-b88a-4ab0-aee1-26e3b32ac9d7/2c066284-8887-41f4-b61e-b40cb8a906fb/77ab04e0-ca17-45de-8f43-d4b5585142b1"
+					(reference "D23")
 					(unit 1)
 				)
@@
 		(dnp no)
 		(fields_autoplaced yes)
-		(property "Reference" "J14"
+		(property "Reference" "J13"
 			(at 187.96 69.85 0)
 			(effects
@@
 			)
 		)
-		(property "Footprint" "TerminalBlock:TerminalBlock_bornier-8_P5.08mm"
+		(property "Footprint" "SpiritBoi_Footprint_Library:TerminalBlock-Horz-THT-8P-P5.08mm-KF2EDG_Pluggable"
 			(at 187.96 83.82 0)
 			(effects
@@
 			(project "DongTamV2"
 				(path "/2303d546-b88a-4ab0-aee1-26e3b32ac9d7/2c066284-8887-41f4-b61e-b40cb8a906fb/0f07157a-883c-4ea4-935e-e968b282f133"
+					(reference "J13")
+					(unit 1)
+				)
+				(path "/2303d546-b88a-4ab0-aee1-26e3b32ac9d7/2c066284-8887-41f4-b61e-b40cb8a906fb/64421711-110b-460c-9945-866904db2698"
 					(reference "J14")
 					(unit 1)
 				)
-				(path "/2303d546-b88a-4ab0-aee1-26e3b32ac9d7/2c066284-8887-41f4-b61e-b40cb8a906fb/64421711-110b-460c-9945-866904db2698"
+				(path "/2303d546-b88a-4ab0-aee1-26e3b32ac9d7/2c066284-8887-41f4-b61e-b40cb8a906fb/2f9aecb0-00e3-4033-a162-064bbf4c14dd"
 					(reference "J15")
 					(unit 1)
 				)
-				(path "/2303d546-b88a-4ab0-aee1-26e3b32ac9d7/2c066284-8887-41f4-b61e-b40cb8a906fb/2f9aecb0-00e3-4033-a162-064bbf4c14dd"
+				(path "/2303d546-b88a-4ab0-aee1-26e3b32ac9d7/2c066284-8887-41f4-b61e-b40cb8a906fb/77ab04e0-ca17-45de-8f43-d4b5585142b1"
 					(reference "J16")
-					(unit 1)
-				)
-				(path "/2303d546-b88a-4ab0-aee1-26e3b32ac9d7/2c066284-8887-41f4-b61e-b40cb8a906fb/77ab04e0-ca17-45de-8f43-d4b5585142b1"
-					(reference "J17")
 					(unit 1)
 				)
@@
 		(on_board yes)
 		(dnp no)
-		(property "Reference" "D10"
+		(property "Reference" "D12"
 			(at 74.93 158.7499 90)
 			(effects
@@
 			(project "DongTamV2"
 				(path "/2303d546-b88a-4ab0-aee1-26e3b32ac9d7/2c066284-8887-41f4-b61e-b40cb8a906fb/0f07157a-883c-4ea4-935e-e968b282f133"
-					(reference "D10")
-					(unit 1)
-				)
-				(path "/2303d546-b88a-4ab0-aee1-26e3b32ac9d7/2c066284-8887-41f4-b61e-b40cb8a906fb/64421711-110b-460c-9945-866904db2698"
-					(reference "D14")
-					(unit 1)
-				)
-				(path "/2303d546-b88a-4ab0-aee1-26e3b32ac9d7/2c066284-8887-41f4-b61e-b40cb8a906fb/2f9aecb0-00e3-4033-a162-064bbf4c14dd"
-					(reference "D18")
-					(unit 1)
-				)
-				(path "/2303d546-b88a-4ab0-aee1-26e3b32ac9d7/2c066284-8887-41f4-b61e-b40cb8a906fb/77ab04e0-ca17-45de-8f43-d4b5585142b1"
-					(reference "D22")
+					(reference "D12")
+					(unit 1)
+				)
+				(path "/2303d546-b88a-4ab0-aee1-26e3b32ac9d7/2c066284-8887-41f4-b61e-b40cb8a906fb/64421711-110b-460c-9945-866904db2698"
+					(reference "D16")
+					(unit 1)
+				)
+				(path "/2303d546-b88a-4ab0-aee1-26e3b32ac9d7/2c066284-8887-41f4-b61e-b40cb8a906fb/2f9aecb0-00e3-4033-a162-064bbf4c14dd"
+					(reference "D20")
+					(unit 1)
+				)
+				(path "/2303d546-b88a-4ab0-aee1-26e3b32ac9d7/2c066284-8887-41f4-b61e-b40cb8a906fb/77ab04e0-ca17-45de-8f43-d4b5585142b1"
+					(reference "D24")
 					(unit 1)
 				)
@@
 		(dnp no)
 		(fields_autoplaced yes)
-		(property "Reference" "D7"
+		(property "Reference" "D9"
 			(at 74.93 24.1299 90)
 			(effects
@@
 			(project "DongTamV2"
 				(path "/2303d546-b88a-4ab0-aee1-26e3b32ac9d7/2c066284-8887-41f4-b61e-b40cb8a906fb/0f07157a-883c-4ea4-935e-e968b282f133"
-					(reference "D7")
-					(unit 1)
-				)
-				(path "/2303d546-b88a-4ab0-aee1-26e3b32ac9d7/2c066284-8887-41f4-b61e-b40cb8a906fb/64421711-110b-460c-9945-866904db2698"
-					(reference "D11")
-					(unit 1)
-				)
-				(path "/2303d546-b88a-4ab0-aee1-26e3b32ac9d7/2c066284-8887-41f4-b61e-b40cb8a906fb/2f9aecb0-00e3-4033-a162-064bbf4c14dd"
-					(reference "D15")
-					(unit 1)
-				)
-				(path "/2303d546-b88a-4ab0-aee1-26e3b32ac9d7/2c066284-8887-41f4-b61e-b40cb8a906fb/77ab04e0-ca17-45de-8f43-d4b5585142b1"
-					(reference "D19")
+					(reference "D9")
+					(unit 1)
+				)
+				(path "/2303d546-b88a-4ab0-aee1-26e3b32ac9d7/2c066284-8887-41f4-b61e-b40cb8a906fb/64421711-110b-460c-9945-866904db2698"
+					(reference "D13")
+					(unit 1)
+				)
+				(path "/2303d546-b88a-4ab0-aee1-26e3b32ac9d7/2c066284-8887-41f4-b61e-b40cb8a906fb/2f9aecb0-00e3-4033-a162-064bbf4c14dd"
+					(reference "D17")
+					(unit 1)
+				)
+				(path "/2303d546-b88a-4ab0-aee1-26e3b32ac9d7/2c066284-8887-41f4-b61e-b40cb8a906fb/77ab04e0-ca17-45de-8f43-d4b5585142b1"
+					(reference "D21")
 					(unit 1)
 				)
@@
 		(dnp no)
 		(fields_autoplaced yes)
-		(property "Reference" "D8"
+		(property "Reference" "D10"
 			(at 74.93 69.8499 90)
 			(effects
@@
 			(project "DongTamV2"
 				(path "/2303d546-b88a-4ab0-aee1-26e3b32ac9d7/2c066284-8887-41f4-b61e-b40cb8a906fb/0f07157a-883c-4ea4-935e-e968b282f133"
-					(reference "D8")
-					(unit 1)
-				)
-				(path "/2303d546-b88a-4ab0-aee1-26e3b32ac9d7/2c066284-8887-41f4-b61e-b40cb8a906fb/64421711-110b-460c-9945-866904db2698"
-					(reference "D12")
-					(unit 1)
-				)
-				(path "/2303d546-b88a-4ab0-aee1-26e3b32ac9d7/2c066284-8887-41f4-b61e-b40cb8a906fb/2f9aecb0-00e3-4033-a162-064bbf4c14dd"
-					(reference "D16")
-					(unit 1)
-				)
-				(path "/2303d546-b88a-4ab0-aee1-26e3b32ac9d7/2c066284-8887-41f4-b61e-b40cb8a906fb/77ab04e0-ca17-45de-8f43-d4b5585142b1"
-					(reference "D20")
-					(unit 1)
-				)
+					(reference "D10")
+					(unit 1)
+				)
+				(path "/2303d546-b88a-4ab0-aee1-26e3b32ac9d7/2c066284-8887-41f4-b61e-b40cb8a906fb/64421711-110b-460c-9945-866904db2698"
+					(reference "D14")
+					(unit 1)
+				)
+				(path "/2303d546-b88a-4ab0-aee1-26e3b32ac9d7/2c066284-8887-41f4-b61e-b40cb8a906fb/2f9aecb0-00e3-4033-a162-064bbf4c14dd"
+					(reference "D18")
+					(unit 1)
+				)
+				(path "/2303d546-b88a-4ab0-aee1-26e3b32ac9d7/2c066284-8887-41f4-b61e-b40cb8a906fb/77ab04e0-ca17-45de-8f43-d4b5585142b1"
+					(reference "D22")
+					(unit 1)
+				)

Commit message: layout p1
Connections:
- net VAN2-: now also J13.4 (Pin_4); no longer J13.6 (Pin_6)
- net VAN3-: now also J13.6 (Pin_6); no longer J13.4 (Pin_4)
Changed lines of the file:
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@@
+	)
+	(label "VAN2-"
+		(at 182.88 83.82 180)
+		(fields_autoplaced yes)
+		(effects
+			(font
+				(size 1.27 1.27)
+			)
+			(justify right bottom)
+		)
 	)
 	(label "VAN2-"
@@
 		)
 	)
-	(label "VAN2-"
-		(at 182.88 88.9 180)
-		(fields_autoplaced yes)
-		(effects
-			(font
-				(size 1.27 1.27)
-			)
-			(justify right bottom)
-		)
-	)
 	(label "VAN4+"
 		(at 55.88 158.75 0)
@@
 		)
 	)
+	(label "VAN3+"
+		(at 182.88 86.36 180)
+		(fields_autoplaced yes)
+		(effects
+			(font
+				(size 1.27 1.27)
+			)
+			(justify right bottom)
+		)
+	)
 	(label "VAN4-"
 		(at 182.88 93.98 180)
@@
 		)
 	)
+	(label "VAN3-"
+		(at 182.88 88.9 180)
+		(fields_autoplaced yes)
+		(effects
+			(font
+				(size 1.27 1.27)
+			)
+			(justify right bottom)
+		)
+	)
 	(label "VAN2+"
 		(at 182.88 81.28 180)
@@
 		)
 	)
-	(label "VAN3-"
-		(at 182.88 83.82 180)
-		(fields_autoplaced yes)
-		(effects
-			(font
-				(size 1.27 1.27)
-			)
-			(justify right bottom)
-		)
-	)
 	(label "VAN1-"
 		(at 58.42 26.67 0)
@@
 		)
 	)
-	(label "VAN3+"
-		(at 182.88 86.36 180)
-		(fields_autoplaced yes)
-		(effects
-			(font
-				(size 1.27 1.27)
-			)
-			(justify right bottom)
-		)
-	)

Commit message: Layout p2, fix Analog VCC and GND for opamp circuit
Connections:
- net +5V renamed AnalogVCC
- net GND renamed AnalogGND

Commit message: Complete layout, HW685 not layout yet
Connections:
- net AnalogGND: no longer R54.2, R55.2, R56.2, R57.2, R58.2, R59.2, R60.2, R61.2
- new net GND: R54.2, R55.2, R56.2, R57.2, R58.2, R59.2, R60.2, R61.2

Commit message: fix: name 1N4007 to 1N4148W
Parts:
- D10, D11, D12, D9: value 1N4007 -> 1N4148W
Changed lines of the file:
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@@
 			)
 		)
-		(property "Value" "1N4007"
+		(property "Value" "1N4148W"
 			(at 74.93 119.3799 90)
 			(effects
@@
 			)
 		)
-		(property "Value" "1N4007"
+		(property "Value" "1N4148W"
 			(at 74.93 161.2899 90)
 			(effects
@@
 			)
 		)
-		(property "Value" "1N4007"
+		(property "Value" "1N4148W"
 			(at 74.93 26.6699 90)
 			(effects
@@
 			)
 		)
-		(property "Value" "1N4007"
+		(property "Value" "1N4148W"
 			(at 74.93 72.3899 90)
 			(effects
